File: penvmon/penvmon.sch (EAGLE design)
At the start: 20 parts, among them IC2 7805TV, U1 ZC563900

Commit message: vibha_layout_done
kindly check the layout once
Parts:
- removed JP3: (no value), jumper:JP1E
- removed LDR: 10k, adafruit:R-US_M0805
Connections:
- removed net DOWN: JP2.7, NANO.D6
- removed net LDR_SIG: JP1.12, JP3.2, LDR.1, NANO.A0
- new net 12: JP1.12, NANO.A0
- net 5V: no longer JP3.1
- net BACK: now also J1.4, JP2.7, NANO.D6; no longer J1.6
- net DOWN(NA): now also J1.7; no longer J1.4
- net GND: no longer LDR.2
- net OK: now also J1.6; no longer J1.7
Changed lines of the file:
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@@
 <part name="I2C_DISP" library="jumper" library_urn="urn:adsk.eagle:library:252" deviceset="JP4E" device="" package3d_urn="urn:adsk.eagle:package:15463/1"/>
 <part name="DHT11" library="jumper" library_urn="urn:adsk.eagle:library:252" deviceset="JP4E" device="" package3d_urn="urn:adsk.eagle:package:15463/1"/>
-<part name="LDR" library="adafruit" library_urn="urn:adsk.eagle:library:420" deviceset="R-US_" device="M0805" package3d_urn="urn:adsk.eagle:package:6240587/1" value="10k"/>
-<part name="JP3" library="jumper" library_urn="urn:adsk.eagle:library:252" deviceset="JP1E" device="" package3d_urn="urn:adsk.eagle:package:15455/1"/>
 <part name="MPU6050" library="con-lsta" library_urn="urn:adsk.eagle:library:161" deviceset="FE08-1" device="" package3d_urn="urn:adsk.eagle:package:8194/1"/>
 </parts>
@@
 <attribute name="VALUE" x="223.52" y="84.455" size="1.778" layer="96" rot="R180"/>
 </instance>
-<instance part="LDR" gate="G$1" x="222.758" y="51.308" smashed="yes" rot="R270">
-<attribute name="NAME" x="224.2566" y="55.118" size="1.778" layer="95" rot="R270"/>
-<attribute name="VALUE" x="219.456" y="55.118" size="1.778" layer="96" rot="R270"/>
-</instance>
-<instance part="JP3" gate="A" x="226.06" y="60.96" smashed="yes" rot="R270">
-<attribute name="NAME" x="226.06" y="62.23" size="1.778" layer="95"/>
-<attribute name="VALUE" x="226.06" y="55.245" size="1.778" layer="96"/>
-</instance>
 <instance part="MPU6050" gate="G$1" x="223.012" y="19.812" smashed="yes">
 <attribute name="VALUE" x="221.742" y="7.112" size="1.778" layer="96"/>
@@
 </segment>
 <segment>
-<pinref part="LDR" gate="G$1" pin="2"/>
-<wire x1="222.758" y1="46.228" x2="222.758" y2="43.18" width="0.1524" layer="91"/>
-<wire x1="222.758" y1="43.18" x2="223.52" y2="43.18" width="0.1524" layer="91"/>
-<label x="223.52" y="43.18" size="1.778" layer="95"/>
-</segment>
-<segment>
 <pinref part="MPU6050" gate="G$1" pin="7"/>
 <wire x1="230.632" y1="27.432" x2="245.872" y2="27.432" width="0.1524" layer="91"/>
@@
 </segment>
 </net>
-<net name="DOWN" class="0">
-<segment>
-<pinref part="NANO" gate="G$1" pin="D6"/>
-<wire x1="105.664" y1="71.628" x2="91.186" y2="71.628" width="0.1524" layer="91"/>
-<pinref part="JP2" gate="A" pin="7"/>
-<label x="98.044" y="71.628" size="1.778" layer="95"/>
-</segment>
-</net>
 <net name="RIGHT" class="0">
 <segment>
@@
 </segment>
 <segment>
-<pinref part="JP3" gate="A" pin="1"/>
-<wire x1="223.52" y1="60.96" x2="215.9" y2="60.96" width="0.1524" layer="91"/>
-<wire x1="215.9" y1="60.96" x2="215.9" y2="63.5" width="0.1524" layer="91"/>
-<label x="215.9" y="63.5" size="1.778" layer="95"/>
-</segment>
-<segment>
 <pinref part="MPU6050" gate="G$1" pin="8"/>
 <wire x1="230.632" y1="29.972" x2="245.872" y2="29.972" width="0.1524" layer="91"/>
@@
 <net name="OK" class="0">
 <segment>
-<pinref part="J1" gate="G$1" pin="7"/>
-<wire x1="280.924" y1="5.588" x2="286.004" y2="5.588" width="0.1524" layer="91"/>
-<label x="283.464" y="5.588" size="1.778" layer="95"/>
-</segment>
-<segment>
 <pinref part="NANO" gate="G$1" pin="D5"/>
 <wire x1="105.664" y1="74.168" x2="91.186" y2="74.168" width="0.1524" layer="91"/>
@@
 <label x="98.044" y="74.168" size="1.778" layer="95"/>
 </segment>
+<segment>
+<pinref part="J1" gate="G$1" pin="6"/>
+<wire x1="270.764" y1="3.048" x2="263.144" y2="3.048" width="0.1524" layer="91"/>
+<label x="263.144" y="3.048" size="1.778" layer="95"/>
+</segment>
 </net>
 <net name="LEFT" class="0">
@@
 <net name="BACK" class="0">
 <segment>
-<pinref part="J1" gate="G$1" pin="6"/>
-<wire x1="270.764" y1="3.048" x2="263.144" y2="3.048" width="0.1524" layer="91"/>
-<label x="263.144" y="3.048" size="1.778" layer="95"/>
+<pinref part="NANO" gate="G$1" pin="D6"/>
+<wire x1="105.664" y1="71.628" x2="91.186" y2="71.628" width="0.1524" layer="91"/>
+<pinref part="JP2" gate="A" pin="7"/>
+<label x="98.044" y="71.628" size="1.778" layer="95"/>
+</segment>
+<segment>
+<pinref part="J1" gate="G$1" pin="4"/>
+<wire x1="270.764" y1="0.508" x2="263.144" y2="0.508" width="0.1524" layer="91"/>
+<label x="258.064" y="0.508" size="1.778" layer="95"/>
 </segment>
 </net>
@@
 <net name="DOWN(NA)" class="0">
 <segment>
-<pinref part="J1" gate="G$1" pin="4"/>
-<wire x1="270.764" y1="0.508" x2="263.144" y2="0.508" width="0.1524" layer="91"/>
-<label x="258.064" y="0.508" size="1.778" layer="95"/>
+<pinref part="J1" gate="G$1" pin="7"/>
+<wire x1="280.924" y1="5.588" x2="286.004" y2="5.588" width="0.1524" layer="91"/>
+<label x="283.464" y="5.588" size="1.778" layer="95"/>
 </segment>
 </net>
@@
 </segment>
 </net>
-<net name="LDR_SIG" class="0">
-<segment>
-<pinref part="JP3" gate="A" pin="2"/>
-<pinref part="LDR" gate="G$1" pin="1"/>
-<wire x1="223.52" y1="58.42" x2="222.758" y2="58.42" width="0.1524" layer="91"/>
-<wire x1="222.758" y1="58.42" x2="222.758" y2="56.388" width="0.1524" layer="91"/>
-<wire x1="223.52" y1="58.42" x2="215.9" y2="58.42" width="0.1524" layer="91"/>
-<junction x="223.52" y="58.42"/>
-<label x="213.36" y="58.42" size="1.778" layer="95"/>
-</segment>
+<net name="12" class="0">
 <segment>
 <pinref part="NANO" gate="G$1" pin="A0"/>

Commit message: just_a_little_correction_vibha_project
all the sensors are added and designed
Parts:
- added SOIL_MOI: (no value), jumper:JP4E
Connections:
- removed net A7: JP1.5, NANO.A7
- new net SOIL_A0: JP1.5, NANO.A7, SOIL_MOI.4
- new net SOIL_D0: SOIL_MOI.3
- net 5V: now also SOIL_MOI.1
- net GND: now also SOIL_MOI.2
Changed lines of the file:
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@@
 <part name="DHT11" library="jumper" library_urn="urn:adsk.eagle:library:252" deviceset="JP4E" device="" package3d_urn="urn:adsk.eagle:package:15463/1"/>
 <part name="MPU6050" library="con-lsta" library_urn="urn:adsk.eagle:library:161" deviceset="FE08-1" device="" package3d_urn="urn:adsk.eagle:package:8194/1"/>
+<part name="SOIL_MOI" library="jumper" library_urn="urn:adsk.eagle:library:252" deviceset="JP4E" device="" package3d_urn="urn:adsk.eagle:package:15463/1"/>
 </parts>
 <sheets>
@@
 <attribute name="VALUE" x="221.742" y="7.112" size="1.778" layer="96"/>
 <attribute name="NAME" x="221.742" y="33.274" size="1.778" layer="95"/>
+</instance>
+<instance part="SOIL_MOI" gate="G$1" x="193.548" y="-12.446" smashed="yes" rot="R270">
+<attribute name="NAME" x="186.944" y="-8.636" size="1.778" layer="95"/>
+<attribute name="VALUE" x="193.548" y="-20.701" size="1.778" layer="96"/>
 </instance>
 </instances>
@@
 <label x="231.14" y="96.52" size="1.778" layer="95"/>
 </segment>
+<segment>
+<pinref part="SOIL_MOI" gate="G$1" pin="2"/>
+<wire x1="191.008" y1="-12.446" x2="180.34" y2="-12.446" width="0.1524" layer="91"/>
+<wire x1="180.34" y1="-12.446" x2="180.34" y2="-12.7" width="0.1524" layer="91"/>
+<label x="177.8" y="-12.7" size="1.778" layer="95"/>
+</segment>
 </net>
 <net name="SCK" class="0">
@@
 </segment>
 </net>
-<net name="A7" class="0">
-<segment>
-<pinref part="NANO" gate="G$1" pin="A7"/>
-<wire x1="146.304" y1="81.788" x2="163.576" y2="81.788" width="0.1524" layer="91"/>
-<pinref part="JP1" gate="A" pin="5"/>
-<label x="148.844" y="81.788" size="1.778" layer="95"/>
-</segment>
-</net>
 <net name="5V" class="0">
 <segment>
@@
 <label x="231.14" y="99.06" size="1.778" layer="95"/>
 </segment>
+<segment>
+<pinref part="SOIL_MOI" gate="G$1" pin="1"/>
+<wire x1="191.008" y1="-9.906" x2="180.34" y2="-9.906" width="0.1524" layer="91"/>
+<wire x1="180.34" y1="-9.906" x2="180.34" y2="-10.16" width="0.1524" layer="91"/>
+<label x="177.8" y="-10.16" size="1.778" layer="95"/>
+</segment>
 </net>
 <net name="N$2" class="0">
@@
 </segment>
 </net>
+<net name="SOIL_D0" class="0">
+<segment>
+<pinref part="SOIL_MOI" gate="G$1" pin="3"/>
+<wire x1="191.008" y1="-14.986" x2="180.34" y2="-14.986" width="0.1524" layer="91"/>
+<wire x1="180.34" y1="-14.986" x2="180.34" y2="-15.24" width="0.1524" layer="91"/>
+<label x="177.8" y="-15.24" size="1.778" layer="95"/>
+</segment>
+</net>
+<net name="SOIL_A0" class="0">
+<segment>
+<pinref part="SOIL_MOI" gate="G$1" pin="4"/>
+<wire x1="191.008" y1="-17.526" x2="180.34" y2="-17.526" width="0.1524" layer="91"/>
+<wire x1="180.34" y1="-17.526" x2="180.34" y2="-17.78" width="0.1524" layer="91"/>
+<label x="177.8" y="-17.78" size="1.778" layer="95"/>
+</segment>
+<segment>
+<pinref part="NANO" gate="G$1" pin="A7"/>
+<wire x1="146.304" y1="81.788" x2="163.576" y2="81.788" width="0.1524" layer="91"/>
+<pinref part="JP1" gate="A" pin="5"/>
+<label x="148.844" y="81.788" size="1.778" layer="95"/>
+</segment>
+</net>
