File: penvmon/penvmon.sch (EAGLE design)
At the start: 19 parts, among them IC2 7805TV, U1 ZC563900

Commit message: added pcb image
Connections:
- net 5V: now also U1.VIN
Changed lines of the file:
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@@
 <label x="177.8" y="-10.16" size="1.778" layer="95"/>
+</segment>
+<segment>
+<pinref part="U1" gate="G$1" pin="VIN"/>
+<wire x1="10.668" y1="4.572" x2="-7.62" y2="4.572" width="0.1524" layer="91"/>
+<wire x1="-7.62" y1="4.572" x2="-7.62" y2="5.08" width="0.1524" layer="91"/>
+<label x="-5.08" y="5.08" size="1.778" layer="95"/>
 </segment>
 </net>
